File: the_split_keyboard/the_split_keyboard.kicad_sch (KiCad schematic)
At the start: 0 parts

Commit message: 色々追加
Parts:
- added D1, D2, D3, D4: D, keyboard:D3_TH_SMD, symbol Device:D
- added J2: MJ-4PP-9, keyboard:MJ-4PP-9, symbol kbd:MJ-4PP-9
- added SW1, SW2, SW3, SW4: SW_PUSH, kbd:keyswitch_cherrymx_hotswap_1u, symbol kbd:SW_PUSH
- added SW5: SW_PUSH, kbd:ResetSW, symbol kbd:SW_PUSH
- added U1: ProMicro, kbd:ProMicro, symbol kbd:ProMicro
Connections:
- new net: D1.2 (A), SW1.2
- new net: D4.2 (A), SW4.2
- new net: D3.2 (A), SW3.2
- new net: D2.2 (A), SW2.2
- new net GND: J2.C, SW5.2, U1.23 (GND), U1.3 (GND), U1.4 (GND)
- new net VCC: J2.D, U1.21 (VCC)
- new net col0: SW1.1, SW2.1, U1.20 (F4/A3)
- new net col1: SW3.1, SW4.1, U1.19 (F5/A2)
- new net data: J2.B, U1.2 (RX1/D2)
- new net reset: SW5.1, U1.22 (RST)
- new net row0: D1.1 (K), D4.1 (K), U1.7 (4/D4)
- new net row1: D2.1 (K), D3.1 (K), U1.8 (5/C6)
- no-connect marks 0 -> 16

Commit message: update
Parts:
- SW1, SW2, SW3, SW4: footprint kbd:keyswitch_cherrymx_hotswap_1u -> keyboard:MX_Choc_Hotswap
- U1: footprint kbd:ProMicro -> keyboard:ProMicro_v2
Changed lines of the file:
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@@
 			)
 		)
-		(property "Footprint" "kbd:keyswitch_cherrymx_hotswap_1u"
+		(property "Footprint" "keyboard:MX_Choc_Hotswap"
 			(at 124.46 66.04 0)
 			(hide yes)
@@
 			)
 		)
-		(property "Footprint" "kbd:keyswitch_cherrymx_hotswap_1u"
+		(property "Footprint" "keyboard:MX_Choc_Hotswap"
 			(at 147.32 66.04 0)
 			(hide yes)
@@
 			)
 		)
-		(property "Footprint" "kbd:keyswitch_cherrymx_hotswap_1u"
+		(property "Footprint" "keyboard:MX_Choc_Hotswap"
 			(at 147.32 86.36 0)
 			(hide yes)
@@
 			)
 		)
-		(property "Footprint" "kbd:ProMicro"
+		(property "Footprint" "keyboard:ProMicro_v2"
 			(at 58.42 92.71 0)
 			(hide yes)
@@
 			)
 		)
-		(property "Footprint" "kbd:keyswitch_cherrymx_hotswap_1u"
+		(property "Footprint" "keyboard:MX_Choc_Hotswap"
 			(at 124.46 86.36 0)
 			(hide yes)
